Commit message: first working version, just impedance

File: urdf/kr10r1100sixx.urdf (robot description, URDF)
Before this commit: robot kuka_kr10r1100sixx, 9 links, 8 joints
Links:
- removed link tool0
- link link_6: mass 0.01 -> 10.0
Joints:
- removed joint joint_a6-tool0

Commit message: Modify algortim transformation. Modify params.

File: urdf/kr10r1100sixx.urdf (robot description, URDF)
Before this commit: robot kuka_kr10r1100sixx, 8 links, 7 joints
Links:
- link link_6: mass 10.0 -> 20.0

Commit message: first version of tool frame impedance.

File: urdf/kr10r1100sixx.urdf (robot description, URDF)
Before this commit: robot kuka_kr10r1100sixx, 8 links, 7 joints
Links:
- link link_6: mass 20.0 -> 15.0

Commit message: Working params.

File: urdf/kr10r1100sixx.urdf (robot description, URDF)
Before this commit: robot kuka_kr10r1100sixx, 8 links, 7 joints
Links:
- link link_6: mass 15.0 -> 20
